Commit message: Add files via upload

File: rplidar_cartographer/urdf/head_2d.urdf (robot description, URDF)
Before this commit: robot head_2d, 2 links, 1 joints
Links:
- added link imu_link; visual box size=0.05 0.05 0.05
Joints:
- added joint imu_joint: type fixed, parent base_link, child imu_link, origin xyz=0.1 0.1 0.1 rpy=0 0 0

Commit message: Add files via upload

File: rplidar_cartographer/urdf/head_2d.urdf (robot description, URDF)
Before this commit: robot head_2d, 3 links, 2 joints
Links:
- added link odom; visual box size=0.1 0.1 0.1
Joints:
- added joint odom_joint: type fixed, parent odom, child base_link, origin xyz=0 0 0 rpy=0 0 0
